File: Kaufland/pcb1/pcb1.kicad_pcb (KiCad board)
At the start: 2 copper layers, 109.7 x 106.7 mm, 27 parts, among them J1 AudioJack2, J2 Barrel_Jack, Q1 IRLB8721PBF, Q2 IRLB8721PBF, Q3 IRLB8721PBF, Q4 IRLB8721PBF, Q5 IRLB8721PBF, Q6 IRLB8721PBF, SW1 SW_Push, SW2 SW_Push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

Commit message: box v2
Parts:
- moved U2 4.06 mm to (48.8, 121.4)
- moved U3 4.06 mm to (48.8, 138.2)
Routing:
- net +12V: track 131.1 -> 139.5 mm
- net Net-(Q6-Pad3): track 58.2 -> 63.4 mm
- net Net-(Q5-Pad3): track 51.3 -> 55.9 mm
- net Net-(Q4-Pad3): track 41.7 -> 46.2 mm
- net Net-(Q3-Pad3): track 68.1 -> 72.2 mm
- net Net-(Q2-Pad3): track 54.9 -> 58.9 mm
- net Net-(Q1-Pad3): track 37.2 -> 41.3 mm
Changed lines of the file:
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@@
     (thickness 1.6)
     (drawings 12)
-    (tracks 246)
+    (tracks 263)
     (zones 0)
     (modules 27)
@@
   )
   (setup
-    (last_trace_width 0.5)
+    (last_trace_width 0.25)
     (user_trace_width 0.5)
     (trace_clearance 0.2)
@@
   )
   (module Connector_JST:JST_EH_S4B-EH_1x04_P2.50mm_Horizontal (layer F.Cu)
-    (at 52.832 138.176 90)
+    (at 48.768 138.176 90)
     (descr "JST EH series connector, S4B-EH (http://www.jst-mfg.com/product/pdf/eng/eEH.pdf), generated with kicad-footprint-generator")
     (tags "connector JST EH horizontal")
@@
   )
   (module Connector_JST:JST_EH_S4B-EH_1x04_P2.50mm_Horizontal (layer F.Cu)
-    (at 52.832 121.412 90)
+    (at 48.768 121.412 90)
     (descr "JST EH series connector, S4B-EH (http://www.jst-mfg.com/product/pdf/eng/eEH.pdf), generated with kicad-footprint-generator")
     (tags "connector JST EH horizontal")
@@
   (segment (start 57.912 116.332) (end 52.832 121.412) (width 0.5) (layer B.Cu) (net 16))
   (segment (start 57.912 109.22) (end 57.912 116.332) (width 0.5) (layer B.Cu) (net 16))
-  (segment (start 51.857 121.412) (end 50.8 122.469) (width 0.5) (layer B.Cu) (net 16))
   (segment (start 52.832 121.412) (end 51.857 121.412) (width 0.5) (layer B.Cu) (net 16))
-  (segment (start 50.8 122.469) (end 50.8 136.144) (width 0.5) (layer B.Cu) (net 16))
-  (segment (start 50.8 136.144) (end 52.832 138.176) (width 0.5) (layer B.Cu) (net 16))
+  (segment (start 50.759 138.176) (end 52.832 136.103) (width 0.5) (layer F.Cu) (net 16))
+  (segment (start 52.832 124.501) (end 49.743 121.412) (width 0.5) (layer F.Cu) (net 16))
+  (segment (start 49.743 121.412) (end 48.768 121.412) (width 0.5) (layer F.Cu) (net 16))
+  (segment (start 52.832 136.103) (end 52.832 124.501) (width 0.5) (layer F.Cu) (net 16))
+  (segment (start 48.768 121.412) (end 52.832 121.412) (width 0.5) (layer B.Cu) (net 16))
+  (segment (start 50.292 138.176) (end 50.759 138.176) (width 0.5) (layer F.Cu) (net 16))
+  (segment (start 50.292 138.176) (end 48.768 138.176) (width 0.5) (layer F.Cu) (net 16))
+  (segment (start 49.784 138.176) (end 50.292 138.176) (width 0.5) (layer F.Cu) (net 16))
   (segment (start 124.46 123.185) (end 124.46 131.572) (width 0.25) (layer F.Cu) (net 17))
   (segment (start 124.46 121.92) (end 124.46 123.185) (width 0.25) (layer F.Cu) (net 17))
@@
   (via (at 81.788 120.396) (size 0.8) (drill 0.4) (layers F.Cu B.Cu) (net 47))
   (segment (start 81.788 120.396) (end 81.788 128.016) (width 0.25) (layer B.Cu) (net 47))
+  (segment (start 52.832 118.912) (end 48.768 118.912) (width 0.25) (layer F.Cu) (net 47))
   (segment (start 52.832 116.412) (end 61.04 116.412) (width 0.25) (layer F.Cu) (net 48))
   (segment (start 61.04 116.412) (end 61.976 117.348) (width 0.25) (layer F.Cu) (net 48))
@@
   (segment (start 83.82 138.684) (end 84.328 138.176) (width 0.25) (layer B.Cu) (net 48))
   (segment (start 62.992 138.684) (end 83.82 138.684) (width 0.25) (layer B.Cu) (net 48))
+  (segment (start 52.832 116.412) (end 48.768 116.412) (width 0.25) (layer F.Cu) (net 48))
   (segment (start 52.832 113.912) (end 63.112 113.912) (width 0.25) (layer F.Cu) (net 49))
   (segment (start 63.112 113.912) (end 64.008 114.808) (width 0.25) (layer F.Cu) (net 49))
@@
   (segment (start 82.804 148.336) (end 86.868 144.272) (width 0.25) (layer F.Cu) (net 49))
   (segment (start 66.548 148.336) (end 82.804 148.336) (width 0.25) (layer F.Cu) (net 49))
+  (segment (start 52.832 113.912) (end 48.768 113.912) (width 0.25) (layer F.Cu) (net 49))
   (segment (start 52.832 135.676) (end 52.832 135.636) (width 0.25) (layer B.Cu) (net 50))
   (segment (start 58.968 129.54) (end 91.948 129.54) (width 0.25) (layer B.Cu) (net 50))
   (segment (start 52.832 135.676) (end 58.968 129.54) (width 0.25) (layer B.Cu) (net 50))
+  (segment (start 50.252 135.676) (end 48.768 135.676) (width 0.25) (layer B.Cu) (net 50))
+  (segment (start 50.252 135.676) (end 52.832 135.676) (width 0.25) (layer B.Cu) (net 50))
+  (segment (start 49.784 135.676) (end 50.252 135.676) (width 0.25) (layer B.Cu) (net 50))
   (segment (start 100.076 126.492) (end 98.552 124.968) (width 0.25) (layer F.Cu) (net 51))
   (segment (start 98.552 124.968) (end 76.708 124.968) (width 0.25) (layer F.Cu) (net 51))
@@
   (segment (start 61.04 124.968) (end 52.832 133.176) (width 0.25) (layer B.Cu) (net 51))
   (segment (start 76.708 124.968) (end 61.04 124.968) (width 0.25) (layer B.Cu) (net 51))
+  (segment (start 50.372 133.176) (end 48.768 133.176) (width 0.25) (layer B.Cu) (net 51))
+  (segment (start 50.372 133.176) (end 49.784 133.176) (width 0.25) (layer B.Cu) (net 51))
+  (segment (start 52.832 133.176) (end 50.372 133.176) (width 0.25) (layer B.Cu) (net 51))
   (segment (start 108.204 123.952) (end 75.184 123.952) (width 0.25) (layer F.Cu) (net 52))
   (via (at 75.184 123.952) (size 0.8) (drill 0.4) (layers F.Cu B.Cu) (net 52))
   (segment (start 59.556 123.952) (end 52.832 130.676) (width 0.25) (layer B.Cu) (net 52))
   (segment (start 75.184 123.952) (end 59.556 123.952) (width 0.25) (layer B.Cu) (net 52))
+  (segment (start 50.92 130.676) (end 48.768 130.676) (width 0.25) (layer B.Cu) (net 52))
+  (segment (start 50.92 130.676) (end 49.784 130.676) (width 0.25) (layer B.Cu) (net 52))
+  (segment (start 52.832 130.676) (end 50.92 130.676) (width 0.25) (layer B.Cu) (net 52))
 )
