File: Kaufland/pcb1/pcb2/pcb2.sch (KiCad schematic (older format))
At the start: 31 parts, among them J1 Raspberry_Pi_2_3, SW1 SW_Push, SW10 SW_Push, SW11 SW_Push, SW12 SW_Push, SW13 SW_Push, SW14 SW_Push, SW15 SW_Push, SW16 SW_Push, SW17 SW_Push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

Commit message: pcb2 routed
Parts:
- J1: footprint (none) -> pcb1:MODULE_RASPBERRY_PI_3_MODEL_B+
- SW1, SW10, SW11, SW12, SW13, SW14, SW15, SW16, SW17, SW18, SW19, SW2, SW20, SW3, SW4, SW5, SW6, SW7, SW8, SW9: footprint Connector_PinSocket_2.54mm:PinSocket_2x01_P2.54mm_Horizontal -> Connector_PinSocket_2.54mm:PinSocket_2x01_P2.54mm_Vertical
Changed lines of the file:
@@
 F 0 "J1" H 2750 3581 50  0000 C CNN
 F 1 "Raspberry_Pi_2_3" H 2750 3490 50  0000 C CNN
-F 2 "" H 2750 2100 50  0001 C CNN
+F 2 "pcb1:MODULE_RASPBERRY_PI_3_MODEL_B+" H 2750 2100 50  0001 C CNN
 F 3 "https://www.raspberrypi.org/documentation/hardware/raspberrypi/schematics/rpi_SCH_3bplus_1p0_reduced.pdf" H 2750 2100 50  0001 C CNN
 	1    2750 2100
@@
 F 0 "SW1" H 1600 4985 50  0000 C CNN
 F 1 "SW_Push" H 1600 4894 50  0000 C CNN
-F 2 "Connector_PinSocket_2.54mm:PinSocket_2x01_P2.54mm_Horizontal" H 1600 4900 50  0001 C CNN
+F 2 "Connector_PinSocket_2.54mm:PinSocket_2x01_P2.54mm_Vertical" H 1600 4900 50  0001 C CNN
 F 3 "~" H 1600 4900 50  0001 C CNN
 	1    1600 4700
@@
 F 0 "SW5" H 2600 4985 50  0000 C CNN
 F 1 "SW_Push" H 2600 4894 50  0000 C CNN
-F 2 "Connector_PinSocket_2.54mm:PinSocket_2x01_P2.54mm_Horizontal" H 2600 4900 50  0001 C CNN
+F 2 "Connector_PinSocket_2.54mm:PinSocket_2x01_P2.54mm_Vertical" H 2600 4900 50  0001 C CNN
 F 3 "~" H 2600 4900 50  0001 C CNN
 	1    2600 4700
@@
 F 0 "SW9" H 3550 4985 50  0000 C CNN
 F 1 "SW_Push" H 3550 4894 50  0000 C CNN
-F 2 "Connector_PinSocket_2.54mm:PinSocket_2x01_P2.54mm_Horizontal" H 3550 4900 50  0001 C CNN
+F 2 "Connector_PinSocket_2.54mm:PinSocket_2x01_P2.54mm_Vertical" H 3550 4900 50  0001 C CNN
 F 3 "~" H 3550 4900 50  0001 C CNN
 	1    3550 4700
@@
 F 0 "SW13" H 4550 4985 50  0000 C CNN
 F 1 "SW_Push" H 4550 4894 50  0000 C CNN
-F 2 "Connector_PinSocket_2.54mm:PinSocket_2x01_P2.54mm_Horizontal" H 4550 4900 50  0001 C CNN
+F 2 "Connector_PinSocket_2.54mm:PinSocket_2x01_P2.54mm_Vertical" H 4550 4900 50  0001 C CNN
 F 3 "~" H 4550 4900 50  0001 C CNN
 	1    4550 4700
@@
 F 0 "SW17" H 5550 4985 50  0000 C CNN
 F 1 "SW_Push" H 5550 4894 50  0000 C CNN
-F 2 "Connector_PinSocket_2.54mm:PinSocket_2x01_P2.54mm_Horizontal" H 5550 4900 50  0001 C CNN
+F 2 "Connector_PinSocket_2.54mm:PinSocket_2x01_P2.54mm_Vertical" H 5550 4900 50  0001 C CNN
 F 3 "~" H 5550 4900 50  0001 C CNN
 	1    5550 4700
@@
 F 0 "SW18" H 5550 5535 50  0000 C CNN
 F 1 "SW_Push" H 5550 5444 50  0000 C CNN
-F 2 "Connector_PinSocket_2.54mm:PinSocket_2x01_P2.54mm_Horizontal" H 5550 5450 50  0001 C CNN
+F 2 "Connector_PinSocket_2.54mm:PinSocket_2x01_P2.54mm_Vertical" H 5550 5450 50  0001 C CNN
 F 3 "~" H 5550 5450 50  0001 C CNN
 	1    5550 5250
@@
 F 0 "SW14" H 4550 5535 50  0000 C CNN
 F 1 "SW_Push" H 4550 5444 50  0000 C CNN
-F 2 "Connector_PinSocket_2.54mm:PinSocket_2x01_P2.54mm_Horizontal" H 4550 5450 50  0001 C CNN
+F 2 "Connector_PinSocket_2.54mm:PinSocket_2x01_P2.54mm_Vertical" H 4550 5450 50  0001 C CNN
 F 3 "~" H 4550 5450 50  0001 C CNN
 	1    4550 5250
@@
 F 0 "SW10" H 3550 5535 50  0000 C CNN
 F 1 "SW_Push" H 3550 5444 50  0000 C CNN
-F 2 "Connector_PinSocket_2.54mm:PinSocket_2x01_P2.54mm_Horizontal" H 3550 5450 50  0001 C CNN
+F 2 "Connector_PinSocket_2.54mm:PinSocket_2x01_P2.54mm_Vertical" H 3550 5450 50  0001 C CNN
 F 3 "~" H 3550 5450 50  0001 C CNN
 	1    3550 5250
@@
 F 0 "SW6" H 2600 5535 50  0000 C CNN
 F 1 "SW_Push" H 2600 5444 50  0000 C CNN
-F 2 "Connector_PinSocket_2.54mm:PinSocket_2x01_P2.54mm_Horizontal" H 2600 5450 50  0001 C CNN
+F 2 "Connector_PinSocket_2.54mm:PinSocket_2x01_P2.54mm_Vertical" H 2600 5450 50  0001 C CNN
 F 3 "~" H 2600 5450 50  0001 C CNN
 	1    2600 5250
@@
 F 0 "SW2" H 1600 5535 50  0000 C CNN
 F 1 "SW_Push" H 1600 5444 50  0000 C CNN
-F 2 "Connector_PinSocket_2.54mm:PinSocket_2x01_P2.54mm_Horizontal" H 1600 5450 50  0001 C CNN
+F 2 "Connector_PinSocket_2.54mm:PinSocket_2x01_P2.54mm_Vertical" H 1600 5450 50  0001 C CNN
 F 3 "~" H 1600 5450 50  0001 C CNN
 	1    1600 5250
@@
 F 0 "SW3" H 1600 6035 50  0000 C CNN
 F 1 "SW_Push" H 1600 5944 50  0000 C CNN
-F 2 "Connector_PinSocket_2.54mm:PinSocket_2x01_P2.54mm_Horizontal" H 1600 5950 50  0001 C CNN
+F 2 "Connector_PinSocket_2.54mm:PinSocket_2x01_P2.54mm_Vertical" H 1600 5950 50  0001 C CNN
 F 3 "~" H 1600 5950 50  0001 C CNN
 	1    1600 5750
@@
 F 0 "SW7" H 2600 6035 50  0000 C CNN
 F 1 "SW_Push" H 2600 5944 50  0000 C CNN
-F 2 "Connector_PinSocket_2.54mm:PinSocket_2x01_P2.54mm_Horizontal" H 2600 5950 50  0001 C CNN
+F 2 "Connector_PinSocket_2.54mm:PinSocket_2x01_P2.54mm_Vertical" H 2600 5950 50  0001 C CNN
 F 3 "~" H 2600 5950 50  0001 C CNN
 	1    2600 5750
@@
 F 0 "SW11" H 3550 6035 50  0000 C CNN
 F 1 "SW_Push" H 3550 5944 50  0000 C CNN
-F 2 "Connector_PinSocket_2.54mm:PinSocket_2x01_P2.54mm_Horizontal" H 3550 5950 50  0001 C CNN
+F 2 "Connector_PinSocket_2.54mm:PinSocket_2x01_P2.54mm_Vertical" H 3550 5950 50  0001 C CNN
 F 3 "~" H 3550 5950 50  0001 C CNN
 	1    3550 5750
@@
 F 0 "SW15" H 4550 6035 50  0000 C CNN
 F 1 "SW_Push" H 4550 5944 50  0000 C CNN
-F 2 "Connector_PinSocket_2.54mm:PinSocket_2x01_P2.54mm_Horizontal" H 4550 5950 50  0001 C CNN
+F 2 "Connector_PinSocket_2.54mm:PinSocket_2x01_P2.54mm_Vertical" H 4550 5950 50  0001 C CNN
 F 3 "~" H 4550 5950 50  0001 C CNN
 	1    4550 5750
@@
 F 0 "SW19" H 5550 6035 50  0000 C CNN
 F 1 "SW_Push" H 5550 5944 50  0000 C CNN
-F 2 "Connector_PinSocket_2.54mm:PinSocket_2x01_P2.54mm_Horizontal" H 5550 5950 50  0001 C CNN
+F 2 "Connector_PinSocket_2.54mm:PinSocket_2x01_P2.54mm_Vertical" H 5550 5950 50  0001 C CNN
 F 3 "~" H 5550 5950 50  0001 C CNN
 	1    5550 5750
@@
 F 0 "SW4" H 1600 6535 50  0000 C CNN
 F 1 "SW_Push" H 1600 6444 50  0000 C CNN
-F 2 "Connector_PinSocket_2.54mm:PinSocket_2x01_P2.54mm_Horizontal" H 1600 6450 50  0001 C CNN
+F 2 "Connector_PinSocket_2.54mm:PinSocket_2x01_P2.54mm_Vertical" H 1600 6450 50  0001 C CNN
 F 3 "~" H 1600 6450 50  0001 C CNN
 	1    1600 6250
@@
 F 0 "SW8" H 2600 6535 50  0000 C CNN
 F 1 "SW_Push" H 2600 6444 50  0000 C CNN
-F 2 "Connector_PinSocket_2.54mm:PinSocket_2x01_P2.54mm_Horizontal" H 2600 6450 50  0001 C CNN
+F 2 "Connector_PinSocket_2.54mm:PinSocket_2x01_P2.54mm_Vertical" H 2600 6450 50  0001 C CNN
 F 3 "~" H 2600 6450 50  0001 C CNN
 	1    2600 6250
@@
 F 0 "SW12" H 3550 6535 50  0000 C CNN
 F 1 "SW_Push" H 3550 6444 50  0000 C CNN
-F 2 "Connector_PinSocket_2.54mm:PinSocket_2x01_P2.54mm_Horizontal" H 3550 6450 50  0001 C CNN
+F 2 "Connector_PinSocket_2.54mm:PinSocket_2x01_P2.54mm_Vertical" H 3550 6450 50  0001 C CNN
 F 3 "~" H 3550 6450 50  0001 C CNN
 	1    3550 6250
@@
 F 0 "SW16" H 4550 6535 50  0000 C CNN
 F 1 "SW_Push" H 4550 6444 50  0000 C CNN
-F 2 "Connector_PinSocket_2.54mm:PinSocket_2x01_P2.54mm_Horizontal" H 4550 6450 50  0001 C CNN
+F 2 "Connector_PinSocket_2.54mm:PinSocket_2x01_P2.54mm_Vertical" H 4550 6450 50  0001 C CNN
 F 3 "~" H 4550 6450 50  0001 C CNN
 	1    4550 6250
@@
 F 0 "SW20" H 5550 6535 50  0000 C CNN
 F 1 "SW_Push" H 5550 6444 50  0000 C CNN
-F 2 "Connector_PinSocket_2.54mm:PinSocket_2x01_P2.54mm_Horizontal" H 5550 6450 50  0001 C CNN
+F 2 "Connector_PinSocket_2.54mm:PinSocket_2x01_P2.54mm_Vertical" H 5550 6450 50  0001 C CNN
 F 3 "~" H 5550 6450 50  0001 C CNN
 	1    5550 6250
